File: carrier_test/carrier/Drivers.sch (KiCad schematic (older format))
At the start: 5 parts

Commit message: update schematic
Parts:
- removed J? (x2): Conn_01x02, symbol Connector_Generic:Conn_01x02
- added J? (x2): CONN_01x06, symbol agg-kicad:CONN_01x06
- added R? (x4): R, symbol agg-kicad:R
Connections:
- net labels added: ENC1_A, ENC1_B, ENC2_A, ENC2_B
- wire segments 34 -> 66

Commit message: Fix supply, add gps/imu serial, oled
Parts:
- gave numbers to parts that had none: 9
Changed lines of the file:
@@
 $EndDescr
 $Comp
-L Connector:Conn_01x08_Male J?
+L Connector:Conn_01x08_Male J7
 U 1 1 5B5238DA
 P 3400 2500
-F 0 "J?" H 3500 2900 50  0000 C CNN
+F 0 "J7" H 3500 2900 50  0000 C CNN
 F 1 "Conn_01x08_Male" H 3500 3050 50  0000 C CNN
 F 2 "" H 3400 2500 50  0001 C CNN
@@
 $EndComp
 $Comp
-L Connector:Conn_01x08_Male J?
+L Connector:Conn_01x08_Male J6
 U 1 1 5B523949
 P 2700 2500
-F 0 "J?" H 2800 2900 50  0000 R CNN
+F 0 "J6" H 2800 2900 50  0000 R CNN
 F 1 "Conn_01x08_Male" H 3100 3050 50  0000 R CNN
 F 2 "" H 2700 2500 50  0001 C CNN
@@
 $EndComp
 $Comp
-L power:+3.3V #PWR?
+L power:+3.3V #PWR014
 U 1 1 5B524663
 P 1150 2150
-F 0 "#PWR?" H 1150 2000 50  0001 C CNN
+F 0 "#PWR014" H 1150 2000 50  0001 C CNN
 F 1 "+3.3V" H 1165 2323 50  0000 C CNN
 F 2 "" H 1150 2150 50  0001 C CNN
@@
 	1150 2150 1150 2300
 $Comp
-L Device:C C?
+L Device:C C7
 U 1 1 5B5252BC
 P 1150 2500
-F 0 "C?" H 1265 2546 50  0000 L CNN
+F 0 "C7" H 1265 2546 50  0000 L CNN
 F 1 "C" H 1265 2455 50  0000 L CNN
 F 2 "" H 1188 2350 50  0001 C CNN
@@
 Connection ~ 1150 2300
 $Comp
-L power:GND #PWR?
+L power:GND #PWR015
 U 1 1 5B5254DA
 P 1150 2750
-F 0 "#PWR?" H 1150 2500 50  0001 C CNN
+F 0 "#PWR015" H 1150 2500 50  0001 C CNN
 F 1 "GND" H 1155 2577 50  0000 C CNN
 F 2 "" H 1150 2750 50  0001 C CNN
@@
 B1
 $Comp
-L power:+3.3V #PWR?
+L power:+3.3V #PWR018
 U 1 1 5B527271
 P 4600 2050
-F 0 "#PWR?" H 4600 1900 50  0001 C CNN
+F 0 "#PWR018" H 4600 1900 50  0001 C CNN
 F 1 "+3.3V" H 4615 2223 50  0000 C CNN
 F 2 "" H 4600 2050 50  0001 C CNN
@@
 Connection ~ 4600 2200
 $Comp
-L power:GND #PWR?
+L power:GND #PWR017
 U 1 1 5B527C88
 P 3700 3000
-F 0 "#PWR?" H 3700 2750 50  0001 C CNN
+F 0 "#PWR017" H 3700 2750 50  0001 C CNN
 F 1 "GND" H 3705 2827 50  0000 C CNN
 F 2 "" H 3700 3000 50  0001 C CNN
@@
 P 3200 4100
 AR Path="/5B513203/5B4DF0A5" Ref="R?"  Part="1"
-AR Path="/5B5131D9/5B4DF0A5" Ref="R?"  Part="1"
-F 0 "R?" V 3204 4141 50  0000 L CNN
+AR Path="/5B5131D9/5B4DF0A5" Ref="R1"  Part="1"
+F 0 "R1" V 3204 4141 50  0000 L CNN
 F 1 "R" V 3295 4141 50  0000 L CNN
 F 2 "" H 3200 4100 50  0001 C CNN
@@
 P 3400 4100
 AR Path="/5B513203/5B4DF0AC" Ref="R?"  Part="1"
-AR Path="/5B5131D9/5B4DF0AC" Ref="R?"  Part="1"
-F 0 "R?" V 3404 4141 50  0000 L CNN
+AR Path="/5B5131D9/5B4DF0AC" Ref="R2"  Part="1"
+F 0 "R2" V 3404 4141 50  0000 L CNN
 F 1 "R" V 3495 4141 50  0000 L CNN
 F 2 "" H 3400 4100 50  0001 C CNN
@@
 P 3600 4100
 AR Path="/5B513203/5B4DF0B3" Ref="R?"  Part="1"
-AR Path="/5B5131D9/5B4DF0B3" Ref="R?"  Part="1"
-F 0 "R?" V 3604 4141 50  0000 L CNN
+AR Path="/5B5131D9/5B4DF0B3" Ref="R3"  Part="1"
+F 0 "R3" V 3604 4141 50  0000 L CNN
 F 1 "R" V 3695 4141 50  0000 L CNN
 F 2 "" H 3600 4100 50  0001 C CNN
@@
 P 3800 4100
 AR Path="/5B513203/5B4DF0BA" Ref="R?"  Part="1"
-AR Path="/5B5131D9/5B4DF0BA" Ref="R?"  Part="1"
-F 0 "R?" V 3804 4141 50  0000 L CNN
+AR Path="/5B5131D9/5B4DF0BA" Ref="R4"  Part="1"
+F 0 "R4" V 3804 4141 50  0000 L CNN
 F 1 "R" V 3895 4141 50  0000 L CNN
 F 2 "" H 3800 4100 50  0001 C CNN
@@
 	3800 4650 3800 4200
 $Comp
-L agg-kicad:CONN_01x06 J?
+L agg-kicad:CONN_01x06 J8
 U 1 1 5B4DFAA1
 P 6300 2250
-F 0 "J?" H 6223 2041 50  0000 R CNN
+F 0 "J8" H 6223 2041 50  0000 R CNN
 F 1 "CONN_01x06" H 6223 1950 50  0000 R CNN
 F 2 "" H 6300 2250 50  0001 C CNN
@@
 $EndComp
 $Comp
-L agg-kicad:CONN_01x06 J?
+L agg-kicad:CONN_01x06 J9
 U 1 1 5B4E0406
 P 6300 3250
-F 0 "J?" H 6223 3041 50  0000 R CNN
+F 0 "J9" H 6223 3041 50  0000 R CNN
 F 1 "CONN_01x06" H 6223 2950 50  0000 R CNN
 F 2 "" H 6300 3250 50  0001 C CNN
@@
 	5900 2750 6200 2750
 $Comp
-L power:GND #PWR?
+L power:GND #PWR019
 U 1 1 5B4E4E9C
 P 5650 2800
-F 0 "#PWR?" H 5650 2550 50  0001 C CNN
+F 0 "#PWR019" H 5650 2550 50  0001 C CNN
 F 1 "GND" H 5655 2627 50  0000 C CNN
 F 2 "" H 5650 2800 50  0001 C CNN
@@
 $EndComp
 $Comp
-L power:GND #PWR?
+L power:GND #PWR020
 U 1 1 5B4E4EB9
 P 5650 3800
-F 0 "#PWR?" H 5650 3550 50  0001 C CNN
+F 0 "#PWR020" H 5650 3550 50  0001 C CNN
 F 1 "GND" H 5655 3627 50  0000 C CNN
 F 2 "" H 5650 3800 50  0001 C CNN
@@
 	5650 2550 5650 2800
 $Comp
-L power:+3.3V #PWR?
+L power:+3.3V #PWR016
 U 1 1 5B4E5FA9
 P 3600 3800
-F 0 "#PWR?" H 3600 3650 50  0001 C CNN
+F 0 "#PWR016" H 3600 3650 50  0001 C CNN
 F 1 "+3.3V" H 3615 3973 50  0000 C CNN
 F 2 "" H 3600 3800 50  0001 C CNN
@@
 	3600 3800 3600 4000
 $Comp
-L power:+3.3V #PWR?
+L power:+3.3V #PWR021
 U 1 1 5B4E68CD
 P 5750 2000
-F 0 "#PWR?" H 5750 1850 50  0001 C CNN
+F 0 "#PWR021" H 5750 1850 50  0001 C CNN
 F 1 "+3.3V" H 5765 2173 50  0000 C CNN
 F 2 "" H 5750 2000 50  0001 C CNN

Commit message: Updates
Changed lines of the file:
@@
 Text HLabel 3650 2500 2    50   Input ~ 10
 MOT_EN
+Text HLabel 3650 2600 2    50   Input ~ 10
+MOT2_A
 Text HLabel 3650 2700 2    50   Input ~ 10
-MOT2_A
-Text HLabel 3650 2600 2    50   Input ~ 10
 MOT2_B
 Wire Wire Line
