File: baseboard/unav2.sch (KiCad schematic (older format))
At the start: 12 parts, among them J2 Conn_02x24_Odd_Even, J3 IMU, J4 GPS, J5 OLED

Commit message: [UNAV2]
Parts:
- removed C1, C2, C3, C4: C, symbol agg-kicad:C
- removed D1: SCHOTTKY, symbol agg-kicad:SCHOTTKY
- removed J2: Conn_02x24_Odd_Even, symbol Connector_Generic:Conn_02x24_Odd_Even
- added C? (x9): 100nF, Capacitor_SMD:C_0402_1005Metric, symbol Device:C_Small
- added C? (x2): 12p, symbol Device:C_Small
- added C? (x2): 1uF, Capacitor_SMD:C_0402_1005Metric, symbol Device:C_Small
- added C?: C, symbol agg-kicad:C
- added C?: 10n, Capacitor_SMD:C_0402_1005Metric, symbol Device:C_Small
- added C?: 10nF, Capacitor_SMD:C_0402_1005Metric, symbol Device:C_Small
- added C?: 4.7uF, Capacitor_SMD:C_0805_2012Metric, symbol Device:C_Small
- added D?: D_Schottky, symbol Device:D_Schottky
- added D?: BAT54C, symbol Device:D_Schottky_x2_KCom_AAK
- added J?: Micro_SD_Card, symbol Connector:Micro_SD_Card
- added J?: USB_B_Micro, symbol Connector:USB_B_Micro
- added JP?: BOOT, symbol Device:Jumper_NO_Small
- added L?: L_Small, symbol Device:L_Small
- added P?: SWD_TC, agg:TC2030-NL, symbol agg-kicad:SWD_TC
- added R? (x6): 10, Resistor_SMD:R_0402_1005Metric, symbol Device:R_Small
- added R?: 47K, Resistor_SMD:R_0402_1005Metric, symbol Device:R_Small
- added R? (x2): 22, Resistor_SMD:R_0402_1005Metric, symbol Device:R_Small
- added R?: 10K, Resistor_SMD:R_0402_1005Metric, symbol Device:R_Small
- added SW?: Reset, symbol Switch:SW_Push
- added SW?: KEY_UP, symbol Switch:SW_Push
- added SW?: KEY1, symbol Switch:SW_Push
- added SW?: KEY0, symbol Switch:SW_Push
- added Y?: 32.768K, symbol Device:Crystal
- added Y?: 8MHz, symbol Device:Resonator_Small
Connections:
- net labels added: +3.3VA, +5VDD, +5V_EXT, BOOT0, GNDA, NRST, PA1, PA13_SWDIO, PA14_SWCK, PB4_SPI1_MISO, PC12_SDIO_SCK, PC2, PE12, PE13, VBATT, VDDA
- net labels removed: BT0, PA1_ENC3_B, PC12_SDIO_CK, PC2_ADC_MOT3_CUR, PE12_TIM_MOT3_A, PE13_TIM_MOT3_A
- wire segments 172 -> 270
Other:
- note removed: "PB4/SPI1_MISO is \nmissing from header!!!"
- moved on the sheet: C5, C6, J3, J4, J5, U?
