File: baseboard/Power.sch (KiCad schematic (older format))
At the start: 19 parts, among them IC1 BTS6133D, J10 CONN_01x04, Q1 BC817

Commit message: [UNAV2]
Connections:
- net labels added: MAIN_Enable
- net labels removed: MOT_Enable
Changed lines of the file:
@@
 	2350 3100 2350 3000
 Text HLabel 1850 2800 0    50   Input ~ 0
-MOT_Enable
+MAIN_Enable
 $Comp
 L agg-kicad:R R5
